File: _saved_Project 23.sch (KiCad schematic (older format))
At the start: 59 parts, among them J11 SRX 1, J12 SRX 2, J13 SWD, J14 Serial DB, J21 BATT +, J22 BATT-, J61 USB_Micro, J71 Micro_SD_Card_Det, SW11 UI_Btn, SW12 PWR_BTN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

Commit message: Finished sunken micro-usb socket
Parts:
- J11, J12: symbol Project-23-rescue:Conn_02x05_Odd_Even -> Project-23-rescue:Conn_02x05_Odd_Even-Project-23-rescue
- J13: symbol Project-23-rescue:Conn_01x04 -> Project-23-rescue:Conn_01x04-Project-23-rescue
- J61: symbol Project-23-rescue:USB_OTG -> Project-23-rescue:USB_OTG-Project-23-rescue
- SW11, SW12: symbol Project-23-rescue:SW_SPST -> Project-23-rescue:SW_SPST-Project-23-rescue
- U5: symbol Project-23-rescue:Conn_01x07 -> Project-23-rescue:Conn_01x07-Project-23-rescue
Changed lines of the file:
@@
 Rev_Limit
 $Comp
-L Project-23-rescue:Conn_02x05_Odd_Even J11
+L Project-23-rescue:Conn_02x05_Odd_Even-Project-23-rescue J11
 U 1 1 5B049189
 P 2350 9400
@@
 $EndComp
 $Comp
-L Project-23-rescue:Conn_02x05_Odd_Even J12
+L Project-23-rescue:Conn_02x05_Odd_Even-Project-23-rescue J12
 U 1 1 5B049278
 P 2350 10350
@@
 Fwd_Limit
 $Comp
-L Project-23-rescue:SW_SPST SW11
+L Project-23-rescue:SW_SPST-Project-23-rescue SW11
 U 1 1 5B04BEBC
 P 6700 9950
@@
 UI_Btn
 $Comp
-L Project-23-rescue:SW_SPST SW12
+L Project-23-rescue:SW_SPST-Project-23-rescue SW12
 U 1 1 5B04C643
 P 6700 10250
@@
 Power_Btn
 $Comp
-L Project-23-rescue:Conn_01x04 J13
+L Project-23-rescue:Conn_01x04-Project-23-rescue J13
 U 1 1 5B04CC06
 P 5050 10200
@@
 $EndComp
 $Comp
-L Project-23-rescue:Conn_01x07 U5
+L Project-23-rescue:Conn_01x07-Project-23-rescue U5
 U 1 1 5B057DA1
 P 10050 9950
@@
 Pwr_LED
 $Comp
-L Project-23-rescue:USB_OTG J61
+L Project-23-rescue:USB_OTG-Project-23-rescue J61
 U 1 1 5B05AAC7
 P 15500 8750
