File: Project 23.sch (KiCad schematic (older format))
At the start: 65 parts, among them J11 SRX 1, J12 SRX 2, J13 SWD, J21 BATT +, J22 BATT-, J61 USB_Micro, J71 Micro_SD_Card_Det, SW11 UI_Btn, SW12 PWR_BTN, U1 STM32F103C8T7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

Commit message: Reworked USB Socket
Parts:
- removed H1: M2, MountingHole:MountingHole_2.2mm_M2, symbol Mechanical:MountingHole
- J11, J12: symbol Project-23-rescue:Conn_02x05_Odd_Even-Project-23-rescue -> Project-23-rescue:Conn_02x05_Odd_Even-Project-23-rescue-Project-23-rescue
- J13: symbol Project-23-rescue:Conn_01x04-Project-23-rescue -> Project-23-rescue:Conn_01x04-Project-23-rescue-Project-23-rescue
- J61: value USB_Micro -> Molex 0476420001; footprint Project 23:microUsbSunken -> Project 23:Molex0476420001_UsbMicro; symbol Project-23-rescue:USB_OTG-Project-23-rescue -> Project-23-rescue:USB_OTG-Project-23-rescue-Project-23-rescue
- SW11, SW12: symbol Project-23-rescue:SW_SPST-Project-23-rescue -> Project-23-rescue:SW_SPST-Project-23-rescue-Project-23-rescue
- U5: symbol Project-23-rescue:Conn_01x07-Project-23-rescue -> Project-23-rescue:Conn_01x07-Project-23-rescue-Project-23-rescue
Changed lines of the file:
@@
 Rev_Limit
 $Comp
-L Project-23-rescue:Conn_02x05_Odd_Even-Project-23-rescue J11
+L Project-23-rescue:Conn_02x05_Odd_Even-Project-23-rescue-Project-23-rescue J11
 U 1 1 5B049189
 P 2350 9400
@@
 $EndComp
 $Comp
-L Project-23-rescue:Conn_02x05_Odd_Even-Project-23-rescue J12
+L Project-23-rescue:Conn_02x05_Odd_Even-Project-23-rescue-Project-23-rescue J12
 U 1 1 5B049278
 P 2350 10350
@@
 Fwd_Limit
 $Comp
-L Project-23-rescue:SW_SPST-Project-23-rescue SW11
+L Project-23-rescue:SW_SPST-Project-23-rescue-Project-23-rescue SW11
 U 1 1 5B04BEBC
 P 6700 9950
@@
 UI_Btn
 $Comp
-L Project-23-rescue:SW_SPST-Project-23-rescue SW12
+L Project-23-rescue:SW_SPST-Project-23-rescue-Project-23-rescue SW12
 U 1 1 5B04C643
 P 6700 10250
@@
 Power_Btn
 $Comp
-L Project-23-rescue:Conn_01x04-Project-23-rescue J13
+L Project-23-rescue:Conn_01x04-Project-23-rescue-Project-23-rescue J13
 U 1 1 5B04CC06
 P 5050 10200
@@
 $EndComp
 $Comp
-L Project-23-rescue:Conn_01x07-Project-23-rescue U5
+L Project-23-rescue:Conn_01x07-Project-23-rescue-Project-23-rescue U5
 U 1 1 5B057DA1
 P 10050 9950
@@
 Pwr_LED
 $Comp
-L Project-23-rescue:USB_OTG-Project-23-rescue J61
+L Project-23-rescue:USB_OTG-Project-23-rescue-Project-23-rescue J61
 U 1 1 5B05AAC7
 P 15500 8750
-F 0 "J61" H 15300 9200 50  0000 L CNN
-F 1 "USB_Micro" H 15300 9100 50  0000 L CNN
-F 2 "Project 23:microUsbSunken" H 15650 8700 50  0001 C CNN
+F 0 "J61" H 15650 9200 50  0000 L CNN
+F 1 "Molex 0476420001" H 15050 9100 50  0000 L CNN
+F 2 "Project 23:Molex0476420001_UsbMicro" H 15650 8700 50  0001 C CNN
 F 3 "" H 15650 8700 50  0001 C CNN
 	1    15500 8750
@@
 	15350 2700 15550 2700
 $Comp
-L Mechanical:MountingHole H1
-U 1 1 5C0E81B8
-P 9400 7700
-F 0 "H1" H 9500 7746 50  0000 L CNN
-F 1 "M2" H 9500 7655 50  0000 L CNN
-F 2 "MountingHole:MountingHole_2.2mm_M2" H 9400 7700 50  0001 C CNN
-F 3 "~" H 9400 7700 50  0001 C CNN
-	1    9400 7700
-	1    0    0    -1
-$EndComp
-$Comp
 L Mechanical:MountingHole H2

Commit message: Updated SRX connectors
Parts:
- J11, J12: footprint Connector_PinHeader_1.27mm:PinHeader_2x05_P1.27mm_Horizontal -> Project 23:20021512-00010T4LF
Changed lines of the file:
@@
 F 0 "J11" H 2400 9700 50  0000 C CNN
 F 1 "SRX 1" H 2400 9100 50  0000 C CNN
-F 2 "Connector_PinHeader_1.27mm:PinHeader_2x05_P1.27mm_Horizontal" H 2350 9400 50  0001 C CNN
+F 2 "Project 23:20021512-00010T4LF" H 2350 9400 50  0001 C CNN
 F 3 "" H 2350 9400 50  0001 C CNN
 	1    2350 9400
@@
 F 0 "J12" H 2400 10650 50  0000 C CNN
 F 1 "SRX 2" H 2400 10050 50  0000 C CNN
-F 2 "Connector_PinHeader_1.27mm:PinHeader_2x05_P1.27mm_Horizontal" H 2350 10350 50  0001 C CNN
+F 2 "Project 23:20021512-00010T4LF" H 2350 10350 50  0001 C CNN
 F 3 "" H 2350 10350 50  0001 C CNN
 	1    2350 10350
